File: KiCad/TD8/TD8.sch (KiCad schematic (older format))
At the start: 301 parts, among them IC1 CD74HC14, J1 plus_pole, J2 minus_pole, J3 Conn_01x08, J4 Conn_01x08, SW1 DIPSW, SW10 DIPSW, SW11 DIPSW, SW12 DIPSW, SW13 DIPSW, SW14 DIPSW, SW15 DIPSW, SW16 DIPSW, SW17 DIPSW, SW18 DIPSW, SW19 DIPSW, SW2 DIPSW, SW20 DIPSW, SW21 DIPSW, SW22 DIPSW, SW23 DIPSW, SW24 DIPSW, SW25 DIPSW, SW26 DIPSW, SW27 DIPSW, SW28 DIPSW, SW29 Push SW, SW3 DIPSW, SW30 Push SW, SW31 DIPSW, SW32 DIPSW, SW33 SW, SW34 DIPSW, SW35 DIPSW, SW36 SW, SW4 DIPSW, SW5 DIPSW, SW6 DIPSW, SW7 DIPSW, SW8 DIPSW, SW9 DIPSW, U1 74HC154, U10 CD74HC153, U11 CD74HC153, U12 CD74HC153, U13 CD74HC153, U14 CD74HC283, U15 CD74HC283, U16 CD74HC32, U17 CD74HC10, U18 CD74HC540, U19 CD74HC540, U2 CD74HC74, U20 CD74HC14, U3 RegAlow, U4 RegBlow, U5 iolow, U6 pclow, U7 RegAhigh, U8 RegBhigh, U9 iohigh

Commit message: make it easy to work on Pcbnew
Parts:
- removed C10, C11, C12, C13, C14, C15, C16, C17, C18, C2, C22, C23, C24, C3, C4, C5, C6, C7, C8, C9: 0.1μ, Capacitor_THT:C_Disc_D5.0mm_W2.5mm_P5.00mm, symbol Device:C
- removed C19, C20: 10μF 16V, Capacitor_THT:CP_Radial_D5.0mm_P2.50mm, symbol Device:CP
- removed C21: 10μF 16V, Capacitor_THT:CP_Radial_D5.0mm_P2.50mm, symbol Device:C
- removed D1, D10, D100, D101, D102, D103, D104, D105, D106, D107, D108, D109, D11, D110, D111, D112, D113, D114, D115, D116, D117, D118, D119, D12, D120, D121, D122, D123, D124, D125, D126, D127, D128, D129, D13, D130, D131, D132, D133, D134, D135, D136, D137, D138, D139, D14, D140, D141, D142, D143, D144, D145, D146, D147, D148, D149, D15, D150, D151, D152, D153, D154, D155, D156, D157, D158, D159, D16, D160, D161, D162, D163, D164, D165, D166, D167, D168, D169, D17, D170, D171, D172, D173, D174, D175, D176, D177, D178, D179, D18, D180, D181, D182, D183, D184, D185, D186, D187, D188, D189, D19, D190, D191, D192, D2, D20, D21, D22, D23, D24, D25, D26, D27, D28, D29, D3, D30, D31, D32, D33, D34, D35, D36, D37, D38, D39, D4, D40, D41, D42, D43, D44, D45, D46, D47, D48, D49, D5, D50, D51, D52, D53, D54, D55, D56, D57, D58, D59, D6, D60, D61, D62, D63, D64, D65, D66, D67, D68, D69, D7, D70, D71, D72, D73, D74, D75, D76, D77, D78, D79, D8, D80, D81, D82, D83, D84, D85, D86, D87, D88, D89, D9, D90, D91, D92, D93, D94, D95, D96, D97, D98, D99: D, Diode_THT:D_T-1_P5.08mm_Horizontal, symbol Device:D
- removed IC1, U20: CD74HC14, Package_DIP:DIP-14_W10.16mm, symbol CD74HCxx:CD74HC14
- removed J3, J4: Conn_01x08, Connector_PinHeader_2.00mm:PinHeader_1x08_P2.00mm_Vertical, symbol Connector_Generic:Conn_01x08
- removed R10: 33K, Resistor_THT:R_Axial_DIN0204_L3.6mm_D1.6mm_P5.08mm_Horizontal, symbol Device:R
- removed R11, R12: 100, Resistor_THT:R_Axial_DIN0204_L3.6mm_D1.6mm_P5.08mm_Horizontal, symbol Device:R
- removed R13, R14, R15, R16, R17, R18, R19, R20, R21, R22, R23, R24, R4: 10K, Resistor_THT:R_Axial_DIN0204_L3.6mm_D1.6mm_P5.08mm_Horizontal, symbol Device:R
- removed R2, R3: 1K, Resistor_THT:R_Axial_DIN0204_L3.6mm_D1.6mm_P5.08mm_Horizontal, symbol Device:R
- removed R5, R6, R7, R8: 100K, Resistor_THT:R_Axial_DIN0204_L3.6mm_D1.6mm_P5.08mm_Horizontal, symbol Device:R
- removed R9: 3.3K, Resistor_THT:R_Axial_DIN0204_L3.6mm_D1.6mm_P5.08mm_Horizontal, symbol Device:R
- removed SW1, SW10, SW13, SW14, SW17, SW18, SW2, SW21, SW22, SW25, SW26, SW31, SW32, SW5, SW6, SW9: DIPSW, Button_Switch_THT:SW_DIP_SPSTx04_Slide_9.78x12.34mm_W7.62mm_P2.54mm, symbol Switch:SW_DIP_x04
- removed SW11, SW12, SW15, SW16, SW19, SW20, SW23, SW24, SW27, SW28, SW3, SW34, SW35, SW4, SW7, SW8: DIPSW, Button_Switch_THT:SW_DIP_SPSTx08_Slide_9.78x22.5mm_W7.62mm_P2.54mm, symbol Switch:SW_DIP_x08
- removed SW29, SW30: Push SW, symbol Switch:SW_Push
- removed SW33, SW36: SW, symbol Switch:SW_Push_SPDT
- removed U1: 74HC154, Package_DIP:DIP-24_W10.16mm, symbol myLib:74HC154
- removed U10, U11, U12, U13: CD74HC153, Package_DIP:DIP-16_W10.16mm, symbol CD74HCxx:CD74HC153
- removed U14, U15: CD74HC283, Package_DIP:DIP-16_W10.16mm, symbol CD74HCxx:CD74HC283
- removed U16: CD74HC32, Package_DIP:DIP-14_W10.16mm, symbol CD74HCxx:CD74HC32
- removed U17: CD74HC10, Package_DIP:DIP-14_W10.16mm, symbol CD74HCxx:CD74HC10
- removed U18, U19: CD74HC540, symbol CD74HCxx:CD74HC540
- removed U2: CD74HC74, Package_DIP:DIP-14_W10.16mm, symbol CD74HCxx:CD74HC74
- removed U3: RegAlow, Package_DIP:DIP-16_W10.16mm, symbol CD74HCxx:CD74HC161
- removed U4: RegBlow, Package_DIP:DIP-16_W10.16mm, symbol CD74HCxx:CD74HC161
- removed U5: iolow, Package_DIP:DIP-16_W10.16mm, symbol CD74HCxx:CD74HC161
- removed U6: pclow, Package_DIP:DIP-16_W10.16mm, symbol CD74HCxx:CD74HC161
- removed U7: RegAhigh, Package_DIP:DIP-16_W10.16mm, symbol CD74HCxx:CD74HC161
- removed U8: RegBhigh, Package_DIP:DIP-16_W10.16mm, symbol CD74HCxx:CD74HC161
- removed U9: iohigh, Package_DIP:DIP-16_W10.16mm, symbol CD74HCxx:CD74HC161
- R1: footprint Resistor_THT:R_Axial_DIN0204_L3.6mm_D1.6mm_P5.08mm_Horizontal -> Resistor_THT:R_Axial_DIN0207_L6.3mm_D2.5mm_P10.16mm_Horizontal
Connections:
- net labels removed: 10Hz, 1Hz, A0, A1, A2, A3, Address0, Address1, Address10, Address11, Address12, Address13, Address14, Address15, Address2, Address3, Address4, Address5, Address6, Address7, Address8, Address9, CLOCK, D0, D1, D10, D11, D2, D3, D4, D5, D6, D7, D8, D9, DR0, DR1, DR10, DR11, DR12, DR2, DR3, DR4, DR5, DR6, DR7, DR8, DR9, Manual, ManualClock, Normal, RESET, a0, a1, a2, a3, a4, a5, a6, a7, b0, b1, b2, b3, b4, b5, b6, b7, i0, i1, i2, i3, i4, i5, i6, i7, is0, is1, is2, is3, is4, is5, is6, is7, o0, o1, o2, o3, o4, o5, o6, o7, op0, op1, op2, op3, s0, s1, s2, s3, s4, s5, s6, s7
- wire segments 1036 -> 6
- no-connect marks 17 -> 0
Other:
- moved on the sheet: C1, J1, J2, R1

Commit message: latest update
Parts:
- removed C1: 100μF, Capacitor_THT:CP_Radial_Tantal_D6.0mm_P2.50mm, symbol Device:CP
- removed J1: plus_pole, Connector_PinHeader_2.00mm:PinHeader_1x01_P2.00mm_Vertical, symbol Connector_Generic:Conn_01x01
- removed J2: minus_pole, Connector_PinHeader_2.00mm:PinHeader_1x01_P2.00mm_Vertical, symbol Connector_Generic:Conn_01x01
- removed R1: 1K, Resistor_THT:R_Axial_DIN0207_L6.3mm_D2.5mm_P10.16mm_Horizontal, symbol Device:R
Connections:
- net labels removed: GND, VCC
- wire segments 6 -> 0
Changed lines of the file:
@@
 Comment4 ""
 $EndDescr
-$Comp
-L power:VCC #PWR01
-U 1 1 5E32EBE9
-P 3250 1450
-F 0 "#PWR01" H 3250 1300 50  0001 C CNN
-F 1 "VCC" H 3267 1623 50  0000 C CNN
-F 2 "" H 3250 1450 50  0001 C CNN
-F 3 "" H 3250 1450 50  0001 C CNN
-	1    3250 1450
-	1    0    0    -1
-$EndComp
-$Comp
-L Device:R R1
-U 1 1 5E32F4B1
-P 3250 1600
-F 0 "R1" H 3320 1646 50  0000 L CNN
-F 1 "1K" H 3320 1555 50  0000 L CNN
-F 2 "Resistor_THT:R_Axial_DIN0207_L6.3mm_D2.5mm_P10.16mm_Horizontal" V 3180 1600 50  0001 C CNN
-F 3 "~" H 3250 1600 50  0001 C CNN
-	1    3250 1600
-	1    0    0    -1
-$EndComp
-$Comp
-L power:GND #PWR02
-U 1 1 5E3305FD
-P 3250 1750
-F 0 "#PWR02" H 3250 1500 50  0001 C CNN
-F 1 "GND" H 3255 1577 50  0000 C CNN
-F 2 "" H 3250 1750 50  0001 C CNN
-F 3 "" H 3250 1750 50  0001 C CNN
-	1    3250 1750
-	1    0    0    -1
-$EndComp
-Wire Wire Line
-	3250 1450 3550 1450
-Connection ~ 3250 1450
-Connection ~ 3250 1750
-$Comp
-L Device:CP C1
-U 1 1 5E364B19
-P 3550 1600
-F 0 "C1" H 3668 1646 50  0000 L CNN
-F 1 "100μF" H 3668 1555 50  0000 L CNN
-F 2 "Capacitor_THT:CP_Radial_Tantal_D6.0mm_P2.50mm" H 3588 1450 50  0001 C CNN
-F 3 "~" H 3550 1600 50  0001 C CNN
-	1    3550 1600
-	1    0    0    -1
-$EndComp
-Connection ~ 3550 1450
-Connection ~ 3550 1750
-Wire Wire Line
-	3550 1750 3250 1750
-Wire Wire Line
-	3550 1450 3650 1450
-$Comp
-L Connector_Generic:Conn_01x01 J1
-U 1 1 5E37C8B4
-P 3850 1450
-F 0 "J1" H 3930 1492 50  0000 L CNN
-F 1 " plus_pole" H 3930 1401 50  0000 L CNN
-F 2 "Connector_PinHeader_2.00mm:PinHeader_1x01_P2.00mm_Vertical" H 3850 1450 50  0001 C CNN
-F 3 "~" H 3850 1450 50  0001 C CNN
-	1    3850 1450
-	1    0    0    -1
-$EndComp
-Connection ~ 3650 1450
-Wire Wire Line
-	3650 1450 3850 1450
-Wire Wire Line
-	3550 1750 3650 1750
-$Comp
-L Connector_Generic:Conn_01x01 J2
-U 1 1 5E37ECF6
-P 3850 1750
-F 0 "J2" H 3930 1792 50  0000 L CNN
-F 1 "minus_pole" H 3930 1701 50  0000 L CNN
-F 2 "Connector_PinHeader_2.00mm:PinHeader_1x01_P2.00mm_Vertical" H 3850 1750 50  0001 C CNN
-F 3 "~" H 3850 1750 50  0001 C CNN
-	1    3850 1750
-	1    0    0    -1
-$EndComp
-Connection ~ 3650 1750
-Wire Wire Line
-	3650 1750 3850 1750
 $Sheet
 S 5350 2200 1200 1250
