File: KiCad/TD8/Memory/Memory.sch (KiCad schematic (older format))
At the start: 34 parts, among them U18 CD74HC540, U19 CD74HC540, U20 74HC154

Commit message: latest update
Parts:
- added J1: Conn_01x08, Connector_PinSocket_2.00mm:PinSocket_1x08_P2.00mm_Vertical, symbol Connector_Generic:Conn_01x08
- added J2, J3: Conn_01x04, Connector_PinSocket_2.00mm:PinSocket_1x04_P2.00mm_Vertical, symbol Connector_Generic:Conn_01x04
- C1: renamed from C19; value 0.1μ -> 0.1u
- C2: renamed from C20; value 0.1μ -> 0.1u
- C3: renamed from C21; value 0.1μ -> 0.1u
- renumbered R2 to R1, R11 to R10, R12 to R11, R13 to R12, R3 to R2, R4 to R3, R5 to R4, R6 to R5, R7 to R6, R8 to R7, R9 to R8, R10 to R9, U18 to U1, U19 to U2, U20 to U3
Connections:
- net DR0: now also J1.1 (Pin_1)
- net DR1: now also J1.2 (Pin_2)
- net DR10: now also J2.3 (Pin_3)
- net DR11: now also J2.4 (Pin_4)
- net DR2: now also J1.3 (Pin_3)
- net DR3: now also J1.4 (Pin_4)
- net DR4: now also J1.5 (Pin_5)
- net DR5: now also J1.6 (Pin_6)
- net DR6: now also J1.7 (Pin_7)
- net DR7: now also J1.8 (Pin_8)
- net DR8: now also J2.1 (Pin_1)
- net DR9: now also J2.2 (Pin_2)
- net A0 renamed a0
- net a0: now also J3.1 (Pin_1)
- net A1 renamed a1
- net a1: now also J3.2 (Pin_2)
- net A2 renamed a2
- net a2: now also J3.3 (Pin_3)
- net A3 renamed a3
- net a3: now also J3.4 (Pin_4)
