File: KiCad/TD8/Clock/Clock.kicad_pcb (KiCad board)
At the start: 2 copper layers, 27 parts, among them IC1 CD74HC14, J1 CLOCK, J2 RESET, J3 VCCSOCKET, J4 plus_pole, J5 GNDSOCKET, J6 minus_pole, SW1 Push SW, SW2 SW, SW3 SW, SW4 Push SW

Commit message: Memory.sch
Parts:
- removed IC1: CD74HC14, Package_DIP:DIP-14_W10.16mm
- added U1: CD74HC14, Package_DIP:DIP-14_W10.16mm, F.Cu at (106.5, 72.7)
- moved J5 47.7 mm to (157.8, 72.6)
- moved R9 44.0 mm to (133.1, 88.8)
- moved R12 42.7 mm to (133.1, 80.7)
- moved SW1 42.4 mm to (146.5, 73.5)
- moved R11 41.4 mm to (133.1, 76.7)
- moved R3 41.4 mm to (119.8, 76.7)
- moved J6 38.7 mm to (137.6, 98.7)
- moved R10 35.0 mm to (119.8, 96.1)
- moved C1 32.3 mm to (152.2, 92.8)
- moved SW4 32.1 mm to (133.2, 93.8)
- moved J3 32.0 mm to (137.6, 84.8)
- moved C2 31.4 mm to (155.7, 79.7)
- moved C3 28.8 mm to (155.7, 86.3)
- moved C4 28.8 mm to (145.0, 94.6)
- moved R1 28.8 mm to (119.8, 72.6)
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